Commit message: robot v2 inicio

File: src/my_robot_description/urdf/robot.urdf (robot description, URDF)
Before this commit: robot diff_robot, 6 links, 5 joints
Links:
- added link laser
- link base_link: geometry visual box size=0.18 0.20 0.26
Joints:
- added joint laser_joint: type fixed, parent base_link, child laser, origin xyz=-0.05 -0.005 0.13
- joint base_footprint_joint: origin xyz=0 0 0.04 -> xyz=-0.05 0 0.04
- joint caster_joint: origin xyz=0.08 0 -0.04 -> xyz=0.08 0 0.035
- joint imu_joint: origin xyz=-0.08 0 0.06 rpy=0 1.5708 3.14159 -> xyz=-0.035 -0.01 0.22 rpy=0 1.5708 3.14159
- joint left_wheel_joint: origin xyz=-0.06 0.1 -0.04 rpy=-1.5708 0 0 -> xyz=-0.05 0.1 0.04 rpy=-1.5708 0 0
- joint right_wheel_joint: origin xyz=-0.06 -0.1 -0.04 rpy=-1.5708 0 0 -> xyz=-0.05 -0.1 0.04 rpy=-1.5708 0 0

Commit message: rotacion lidar

File: src/my_robot_description/urdf/robot.urdf (robot description, URDF)
Before this commit: robot diff_robot, 7 links, 6 joints
Joints:
- joint laser_joint: origin xyz=-0.05 -0.005 0.13 -> xyz=-0.05 -0.005 0.13 rpy=0 0 0

Commit message: algunos cambios en orientacion lidar

File: src/my_robot_description/urdf/robot.urdf (robot description, URDF)
Before this commit: robot diff_robot, 7 links, 6 joints
Joints:
- joint laser_joint: origin xyz=-0.05 -0.005 0.13 rpy=0 0 0 -> xyz=-0.05 -0.005 0.13 rpy=0 0 1.5708
